File: ws-400.sch (KiCad schematic (older format))
At the start: 30 parts, among them J1 Conn_02x49, J2 LCD, J5 Conn_02x20_Row_Letter_First, SW3 SW_Push, U1 MCP23017_SS, U2 MCP23017_SS, U3 MCP23017_SS, U4 MCP23017_SS, U5 MCP23017_SS, U6 MCP23017_SS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

Commit message: schematic cleanup
Parts:
- C2, C3, C5, C6, C7, C8: value C_Small -> 100n
Other:
- moved on the sheet: C3, C5, C7, C8
Changed lines of the file:
@@
 P 7700 4900
 F 0 "U5" H 7250 5850 50  0000 C CNN
-F 1 "MCP23017_SS" H 7700 6090 50  0000 C CNN
+F 1 "MCP23017_SS" H 8000 5850 50  0000 C CNN
 F 2 "Package_SO:SSOP-28_5.3x10.2mm_P0.65mm" H 7900 3900 50  0001 L CNN
 F 3 "http://ww1.microchip.com/downloads/en/DeviceDoc/20001952C.pdf" H 7900 3800 50  0001 L CNN
@@
 P 4650 5750
 F 0 "U7" H 4200 7200 50  0000 C CNN
-F 1 "ATmega328-AU" H 4650 4070 50  0000 C CNN
+F 1 "ATmega328-AU" H 5050 7200 50  0000 C CNN
 F 2 "Package_QFP:TQFP-32_7x7mm_P0.8mm" H 4650 5750 50  0001 C CIN
 F 3 "http://ww1.microchip.com/downloads/en/DeviceDoc/ATmega328_P%20AVR%20MCU%20with%20picoPower%20Technology%20Data%20Sheet%2040001984A.pdf" H 4650 5750 50  0001 C CNN
@@
 P 5500 2000
 F 0 "U2" H 5050 2950 50  0000 C CNN
-F 1 "MCP23017_SS" H 5500 3190 50  0000 C CNN
+F 1 "MCP23017_SS" H 5800 2950 50  0000 C CNN
 F 2 "Package_SO:SSOP-28_5.3x10.2mm_P0.65mm" H 5700 1000 50  0001 L CNN
 F 3 "http://ww1.microchip.com/downloads/en/DeviceDoc/20001952C.pdf" H 5700 900 50  0001 L CNN
@@
 P 3300 2000
 F 0 "U1" H 2850 2950 50  0000 C CNN
-F 1 "MCP23017_SS" H 3300 3190 50  0000 C CNN
+F 1 "MCP23017_SS" H 3600 2950 50  0000 C CNN
 F 2 "Package_SO:SSOP-28_5.3x10.2mm_P0.65mm" H 3500 1000 50  0001 L CNN
 F 3 "http://ww1.microchip.com/downloads/en/DeviceDoc/20001952C.pdf" H 3500 900 50  0001 L CNN
@@
 P 9600 2000
 F 0 "U4" H 9150 2950 50  0000 C CNN
-F 1 "MCP23017_SS" H 9600 3190 50  0000 C CNN
+F 1 "MCP23017_SS" H 9900 2950 50  0000 C CNN
 F 2 "Package_SO:SSOP-28_5.3x10.2mm_P0.65mm" H 9800 1000 50  0001 L CNN
 F 3 "http://ww1.microchip.com/downloads/en/DeviceDoc/20001952C.pdf" H 9800 900 50  0001 L CNN
@@
 P 7550 2000
 F 0 "U3" H 7100 2950 50  0000 C CNN
-F 1 "MCP23017_SS" H 7550 3190 50  0000 C CNN
+F 1 "MCP23017_SS" H 7850 2950 50  0000 C CNN
 F 2 "Package_SO:SSOP-28_5.3x10.2mm_P0.65mm" H 7750 1000 50  0001 L CNN
 F 3 "http://ww1.microchip.com/downloads/en/DeviceDoc/20001952C.pdf" H 7750 900 50  0001 L CNN
@@
 P 10100 4950
 F 0 "U6" H 9650 5900 50  0000 C CNN
-F 1 "MCP23017_SS" H 10100 6140 50  0000 C CNN
+F 1 "MCP23017_SS" H 10400 5900 50  0000 C CNN
 F 2 "Package_SO:SSOP-28_5.3x10.2mm_P0.65mm" H 10300 3950 50  0001 L CNN
 F 3 "http://ww1.microchip.com/downloads/en/DeviceDoc/20001952C.pdf" H 10300 3850 50  0001 L CNN
@@
 U 1 1 5F103A5B
 P 800 7300
-F 0 "5V1" H 908 7481 50  0000 C CNN
-F 1 "Conn_01x02_Male" H 908 7390 50  0000 C CNN
+F 0 "5V1" H 700 7300 50  0000 C CNN
+F 1 "Conn_01x02_Male" H 800 7400 50  0000 C CNN
 F 2 "Connector_PinHeader_2.54mm:PinHeader_1x02_P2.54mm_Vertical" H 800 7300 50  0001 C CNN
 F 3 "~" H 800 7300 50  0001 C CNN
@@
 $EndComp
 Wire Wire Line
-	1000 7300 1100 7300
-Wire Wire Line
 	1300 7300 1300 7250
 Wire Wire Line
 	1300 7500 1300 7450
 Wire Wire Line
-	1300 7400 1100 7400
+	1300 7400 1250 7400
 Text Label 8400 5000 0    50   ~ 0
 A40
@@
 L power:PWR_FLAG #FLG0101
 U 1 1 5F140568
-P 1100 7300
-F 0 "#FLG0101" H 1100 7375 50  0001 C CNN
-F 1 "PWR_FLAG" H 1100 7473 50  0000 C CNN
-F 2 "" H 1100 7300 50  0001 C CNN
-F 3 "~" H 1100 7300 50  0001 C CNN
-	1    1100 7300
-	1    0    0    -1
-$EndComp
-Connection ~ 1100 7300
-Wire Wire Line
-	1100 7300 1300 7300
+P 1250 7300
+F 0 "#FLG0101" H 1250 7375 50  0001 C CNN
+F 1 "PWR_FLAG" H 1100 7500 50  0000 C CNN
+F 2 "" H 1250 7300 50  0001 C CNN
+F 3 "~" H 1250 7300 50  0001 C CNN
+	1    1250 7300
+	1    0    0    -1
+$EndComp
 $Comp
 L power:PWR_FLAG #FLG0102
 U 1 1 5F140FED
-P 1100 7400
-F 0 "#FLG0102" H 1100 7475 50  0001 C CNN
-F 1 "PWR_FLAG" H 1100 7573 50  0000 C CNN
-F 2 "" H 1100 7400 50  0001 C CNN
-F 3 "~" H 1100 7400 50  0001 C CNN
-	1    1100 7400
+P 1250 7400
+F 0 "#FLG0102" H 1250 7475 50  0001 C CNN
+F 1 "PWR_FLAG" H 1500 7500 50  0000 C CNN
+F 2 "" H 1250 7400 50  0001 C CNN
+F 3 "~" H 1250 7400 50  0001 C CNN
+	1    1250 7400
 	-1   0    0    1
 $EndComp
-Connection ~ 1100 7400
-Wire Wire Line
-	1100 7400 1000 7400
 Wire Wire Line
 	1400 7250 1300 7250
@@
 U 1 1 5F0A1CB5
 P 1400 7350
-F 0 "C1" H 1488 7396 50  0000 L CNN
-F 1 "100u" H 1488 7305 50  0000 L CNN
+F 0 "C1" H 1350 7500 50  0000 L CNN
+F 1 "100u" V 1500 7250 50  0000 L CNN
 F 2 "Capacitor_Tantalum_SMD:CP_EIA-3528-21_Kemet-B_Pad1.50x2.35mm_HandSolder" H 1400 7350 50  0001 C CNN
 F 3 "~" H 1400 7350 50  0001 C CNN
@@
 U 1 1 5F0A2B7D
 P 1600 7350
-F 0 "C2" H 1692 7396 50  0000 L CNN
-F 1 "C_Small" H 1692 7305 50  0000 L CNN
+F 0 "C2" H 1550 7500 50  0000 L CNN
+F 1 "100n" V 1700 7250 50  0000 L CNN
 F 2 "Capacitor_SMD:C_0805_2012Metric_Pad1.15x1.40mm_HandSolder" H 1600 7350 50  0001 C CNN
 F 3 "~" H 1600 7350 50  0001 C CNN
@@
 L Device:C_Small C3
 U 1 1 5F0A35CE
-P 1750 7350
-F 0 "C3" H 1842 7396 50  0000 L CNN
-F 1 "C_Small" H 1842 7305 50  0000 L CNN
-F 2 "Capacitor_SMD:C_0805_2012Metric_Pad1.15x1.40mm_HandSolder" H 1750 7350 50  0001 C CNN
-F 3 "~" H 1750 7350 50  0001 C CNN
-	1    1750 7350
+P 1800 7350
+F 0 "C3" H 1750 7500 50  0000 L CNN
+F 1 "100n" V 1900 7250 50  0000 L CNN
+F 2 "Capacitor_SMD:C_0805_2012Metric_Pad1.15x1.40mm_HandSolder" H 1800 7350 50  0001 C CNN
+F 3 "~" H 1800 7350 50  0001 C CNN
+	1    1800 7350
 	1    0    0    -1
 $EndComp
@@
 L Device:C_Small C5
 U 1 1 5F0A41B0
-P 2050 7350
-F 0 "C5" H 2142 7396 50  0000 L CNN
-F 1 "C_Small" H 2142 7305 50  0000 L CNN
-F 2 "Capacitor_SMD:C_0805_2012Metric_Pad1.15x1.40mm_HandSolder" H 2050 7350 50  0001 C CNN
-F 3 "~" H 2050 7350 50  0001 C CNN
-	1    2050 7350
+P 2000 7350
+F 0 "C5" H 1950 7500 50  0000 L CNN
+F 1 "100n" V 2100 7250 50  0000 L CNN
+F 2 "Capacitor_SMD:C_0805_2012Metric_Pad1.15x1.40mm_HandSolder" H 2000 7350 50  0001 C CNN
+F 3 "~" H 2000 7350 50  0001 C CNN
+	1    2000 7350
 	1    0    0    -1
 $EndComp
@@
 U 1 1 5F0A43A2
 P 2200 7350
-F 0 "C6" H 2292 7396 50  0000 L CNN
-F 1 "C_Small" H 2292 7305 50  0000 L CNN
+F 0 "C6" H 2150 7500 50  0000 L CNN
+F 1 "100n" V 2300 7250 50  0000 L CNN
 F 2 "Capacitor_SMD:C_0805_2012Metric_Pad1.15x1.40mm_HandSolder" H 2200 7350 50  0001 C CNN
 F 3 "~" H 2200 7350 50  0001 C CNN
@@
 	1    0    0    -1
 $EndComp
-$Comp
-L Device:C_Small C7
-U 1 1 5F0A4766
-P 2350 7350
-F 0 "C7" H 2442 7396 50  0000 L CNN
-F 1 "C_Small" H 2442 7305 50  0000 L CNN
-F 2 "Capacitor_SMD:C_0805_2012Metric_Pad1.15x1.40mm_HandSolder" H 2350 7350 50  0001 C CNN
-F 3 "~" H 2350 7350 50  0001 C CNN
-	1    2350 7350
-	1    0    0    -1
-$EndComp
-$Comp
-L Device:C_Small C8
-U 1 1 5F0A4B1D
-P 2500 7350
-F 0 "C8" H 2592 7396 50  0000 L CNN
-F 1 "C_Small" H 2592 7305 50  0000 L CNN
-F 2 "Capacitor_SMD:C_0805_2012Metric_Pad1.15x1.40mm_HandSolder" H 2500 7350 50  0001 C CNN
-F 3 "~" H 2500 7350 50  0001 C CNN
-	1    2500 7350
-	1    0    0    -1
-$EndComp
 Wire Wire Line
 	1400 7250 1600 7250
 Connection ~ 1400 7250
 Connection ~ 1600 7250
-Wire Wire Line
-	1600 7250 1750 7250
-Connection ~ 1750 7250
-Connection ~ 2050 7250
-Wire Wire Line
-	2050 7250 2200 7250
 Connection ~ 2200 7250
-Wire Wire Line
-	2200 7250 2350 7250
-Connection ~ 2350 7250
-Wire Wire Line
-	2350 7250 2500 7250
-Wire Wire Line
-	2500 7450 2350 7450
 Connection ~ 1400 7450
 Connection ~ 1600 7450
 Wire Wire Line
 	1600 7450 1400 7450
-Connection ~ 1750 7450
-Wire Wire Line
-	1750 7450 1600 7450
-Connection ~ 2050 7450
 Connection ~ 2200 7450
-Wire Wire Line
-	2200 7450 2050 7450
-Connection ~ 2350 7450
-Wire Wire Line
-	2350 7450 2200 7450
 NoConn ~ 5250 5250
 NoConn ~ 5250 5450
@@
 NoConn ~ 4050 4850
 Wire Wire Line
-	1750 7250 2050 7250
-Wire Wire Line
-	1750 7450 2050 7450
-Wire Wire Line
 	3900 4550 4050 4550
 $Comp
@@
 F 3 "" H 3900 4750 50  0001 C CNN
 	1    3900 4750
-	1    0    0    -1
-$EndComp
-$Comp
-L Connector_Generic:Conn_02x05_Odd_Even PROG1
-U 1 1 5F120014
-P 1450 6350
-F 0 "PROG1" H 1500 6767 50  0000 C CNN
-F 1 "Conn_02x05_Odd_Even" H 1500 6676 50  0000 C CNN
-F 2 "Connector_PinHeader_2.54mm:PinHeader_2x05_P2.54mm_Vertical" H 1450 6350 50  0001 C CNN
-F 3 "~" H 1450 6350 50  0001 C CNN
-	1    1450 6350
 	1    0    0    -1
 $EndComp
@@
 Wire Wire Line
 	2450 4300 3050 4300
+$Comp
+L Connector_Generic:Conn_02x05_Odd_Even PROG1
+U 1 1 5F120014
+P 1450 6350
+F 0 "PROG1" H 1500 6767 50  0000 C CNN
+F 1 "Conn_02x05_Odd_Even" H 1500 6676 50  0000 C CNN
+F 2 "Connector_PinHeader_2.54mm:PinHeader_2x05_P2.54mm_Vertical" H 1450 6350 50  0001 C CNN
+F 3 "~" H 1450 6350 50  0001 C CNN
+	1    1450 6350
+	1    0    0    -1
+$EndComp
+$Comp
+L Device:C_Small C7
+U 1 1 5F0A4766
+P 2400 7350
+F 0 "C7" H 2350 7500 50  0000 L CNN
+F 1 "100n" V 2500 7250 50  0000 L CNN
+F 2 "Capacitor_SMD:C_0805_2012Metric_Pad1.15x1.40mm_HandSolder" H 2400 7350 50  0001 C CNN
+F 3 "~" H 2400 7350 50  0001 C CNN
+	1    2400 7350
+	1    0    0    -1
+$EndComp
+$Comp
+L Device:C_Small C8
+U 1 1 5F0A4B1D
+P 2600 7350
+F 0 "C8" H 2550 7500 50  0000 L CNN
+F 1 "100n" V 2700 7250 50  0000 L CNN
+F 2 "Capacitor_SMD:C_0805_2012Metric_Pad1.15x1.40mm_HandSolder" H 2600 7350 50  0001 C CNN
+F 3 "~" H 2600 7350 50  0001 C CNN
+	1    2600 7350
+	1    0    0    -1
+$EndComp
+Connection ~ 1800 7250
+Wire Wire Line
+	1800 7250 2000 7250
+Connection ~ 1800 7450
+Wire Wire Line
+	1800 7450 2000 7450
+Wire Wire Line
+	1600 7450 1800 7450
+Connection ~ 2000 7250
+Connection ~ 2000 7450
+Wire Wire Line
+	2000 7250 2200 7250
+Wire Wire Line
+	2000 7450 2200 7450
+Connection ~ 2400 7250
+Connection ~ 2400 7450
+Wire Wire Line
+	2200 7250 2400 7250
+Wire Wire Line
+	2200 7450 2400 7450
+Wire Wire Line
+	1600 7250 1800 7250
+Wire Wire Line
+	2400 7250 2600 7250
+Wire Wire Line
+	2400 7450 2600 7450
+Connection ~ 1250 7400
+Connection ~ 1250 7300
+Wire Wire Line
+	1250 7300 1300 7300
+Wire Wire Line
+	1000 7300 1250 7300
+Wire Wire Line
+	1000 7400 1250 7400
 $EndSCHEMATC
